Commit message: Add ee_fingers link

File: grippers/gripper_tactile.xacro (robot description, xacro)
@@ -111,3 +111,10 @@
   <origin xyz="-0.033 0.023 0.094" rpy="0 0.378 -1.57"/>
 </xacro:sensor_d435i>
+<!-- END EFFECTOR FINGERS -->
+<link name="ee_fingers"> </link>
+<joint name="tool0_ee" type="fixed">
+  <origin xyz="0 0 0.21" rpy="0 0 0"/>
+  <parent link="tool0"/>
+  <child link="ee_fingers"/>
+</joint>
 </robot>
