Commit message: Fixed transformation

File: grippers/gripper_pushing.xacro (robot description, xacro)
@@ -2,5 +2,5 @@
 <robot xmlns:xacro="http://www.ros.org/wiki/xacro" name="wgs32_camera">
     <xacro:property name="deg" value="0.017453293" /> <!--degrees to radians-->
-    <xacro:include filename="$(find gripper_description)/grippers/yaskawa_tactile.xacro"/>
+    <xacro:include filename="$(find gripper_description)/grippers/gripper_tactile.xacro"/>
     <link name="push_extension">
         <inertial>
@@ -10,19 +10,19 @@
         </inertial>
         <visual>
-          <origin xyz="0.031533 0.21556 -0.045445" rpy="0 0 0"/>
+          <origin xyz="0 0 0" rpy="0 0 0"/>
           <geometry>
-            <mesh filename="package://gripper_description/meshes/pusher_ext.stl" scale="0.001 0.001 0.001"/>
+            <mesh filename="file://$(find gripper_description)/meshes/pusher_ext.stl" scale="0.001 0.001 0.001"/>
           </geometry>
           <material name="white1"/>
         </visual>
         <collision>
-          <origin xyz="0.031533 0.21556 -0.045445" rpy="0 0 0"/>
+          <origin xyz="0 0 0" rpy="0 0 0"/>
           <geometry>
-            <mesh filename="package://gripper_description/meshes/pusher_ext.stl" scale="0.001 0.001 0.001"/>
+            <mesh filename="file://$(find gripper_description)/meshes/pusher_ext.stl" scale="0.001 0.001 0.001"/>
           </geometry>
         </collision>
       </link>
       <joint name="tactile_joint_pusher" type="fixed">
-        <origin xyz="-0.001729 -0.072903 -0.001654" rpy="0 0 0"/>
+        <origin xyz="0.00012757793764987647 -0.2859275779376499 0.07637889688249402" rpy="-1.5606521280013759 0.00020384840978560081 0.020189250214579735"/>
         <parent link="tactile_2"/>
         <child link="push_extension"/>

Commit message: Fixed name

File: grippers/gripper_pushing.xacro (robot description, xacro)
@@ -2,5 +2,5 @@
 <robot xmlns:xacro="http://www.ros.org/wiki/xacro" name="wgs32_camera">
     <xacro:property name="deg" value="0.017453293" /> <!--degrees to radians-->
-    <xacro:include filename="$(find gripper_description)/grippers/gripper_tactile.xacro"/>
+    <xacro:include filename="$(find gripper_description_ros2)/grippers/gripper_tactile.xacro"/>
     <link name="push_extension">
         <inertial>
@@ -12,5 +12,5 @@
           <origin xyz="0 0 0" rpy="0 0 0"/>
           <geometry>
-            <mesh filename="file://$(find gripper_description)/meshes/pusher_ext.stl" scale="0.001 0.001 0.001"/>
+            <mesh filename="file://$(find gripper_description_ros2)/meshes/pusher_ext.stl" scale="0.001 0.001 0.001"/>
           </geometry>
           <material name="white1"/>
@@ -19,5 +19,5 @@
           <origin xyz="0 0 0" rpy="0 0 0"/>
           <geometry>
-            <mesh filename="file://$(find gripper_description)/meshes/pusher_ext.stl" scale="0.001 0.001 0.001"/>
+            <mesh filename="file://$(find gripper_description_ros2)/meshes/pusher_ext.stl" scale="0.001 0.001 0.001"/>
           </geometry>
         </collision>

File: grippers/gripper_tactile.xacro (robot description, xacro)
@@ -12,5 +12,5 @@
       <origin xyz="0 0 0" rpy="0 0 0"/>
       <geometry>
-        <mesh filename="file://$(find gripper_description)/meshes/base_link.stl" scale="0.001 0.001 0.001"/>
+        <mesh filename="file://$(find gripper_description_ros2)/meshes/base_link.stl" scale="0.001 0.001 0.001"/>
       </geometry>
       <material name="white1"/>
@@ -19,5 +19,5 @@
       <origin xyz="0 0 0" rpy="0 0 0"/>
       <geometry>
-        <mesh filename="file://$(find gripper_description)/meshes/base_link.stl" scale="0.001 0.001 0.001"/>
+        <mesh filename="file://$(find gripper_description_ros2)/meshes/base_link.stl" scale="0.001 0.001 0.001"/>
       </geometry>
     </collision>
@@ -32,5 +32,5 @@
       <origin xyz="0 0 0" rpy="0 0 0"/>
       <geometry>
-        <mesh filename="file://$(find gripper_description)/meshes/extension_camera_support.stl" scale="0.001 0.001 0.001"/>
+        <mesh filename="file://$(find gripper_description_ros2)/meshes/extension_camera_support.stl" scale="0.001 0.001 0.001"/>
       </geometry>
       <material name="white1"/>
@@ -39,5 +39,5 @@
       <origin xyz="0 0 0" rpy="0 0 0"/>
       <geometry>
-        <mesh filename="file://$(find gripper_description)/meshes/extension_camera_support.stl" scale="0.001 0.001 0.001"/>
+        <mesh filename="file://$(find gripper_description_ros2)/meshes/extension_camera_support.stl" scale="0.001 0.001 0.001"/>
       </geometry>
     </collision>
@@ -52,5 +52,5 @@
       <origin xyz="0 0 0" rpy="0 0 0"/>
       <geometry>
-        <mesh filename="file://$(find gripper_description)/meshes/finger_ext.stl" scale="0.001 0.001 0.001"/>
+        <mesh filename="file://$(find gripper_description_ros2)/meshes/finger_ext.stl" scale="0.001 0.001 0.001"/>
       </geometry>
       <material name="white1"/>
@@ -59,5 +59,5 @@
       <origin xyz="0 0 0" rpy="0 0 0"/>
       <geometry>
-        <mesh filename="file://$(find gripper_description)/meshes/finger_ext.stl" scale="0.001 0.001 0.001"/>
+        <mesh filename="file://$(find gripper_description_ros2)/meshes/finger_ext.stl" scale="0.001 0.001 0.001"/>
       </geometry>
     </collision>
@@ -72,5 +72,5 @@
       <origin xyz="0 0 0" rpy="0 0 0"/>
       <geometry>
-        <mesh filename="file://$(find gripper_description)/meshes/finger_ext.stl" scale="0.001 0.001 0.001"/>
+        <mesh filename="file://$(find gripper_description_ros2)/meshes/finger_ext.stl" scale="0.001 0.001 0.001"/>
       </geometry>
       <material name="white1"/>
@@ -79,5 +79,5 @@
       <origin xyz="0 0 0" rpy="0 0 0"/>
       <geometry>
-        <mesh filename="file://$(find gripper_description)/meshes/finger_ext.stl" scale="0.001 0.001 0.001"/>
+        <mesh filename="file://$(find gripper_description_ros2)/meshes/finger_ext.stl" scale="0.001 0.001 0.001"/>
       </geometry>
     </collision>
@@ -98,7 +98,7 @@
     <child link="ext_finger_2"/>
   </joint>
-  <xacro:include filename="$(find wsg32_description)/grippers/wsg32.urdf"/>
+  <xacro:include filename="$(find wsg32_description_ros2)/grippers/wsg32.urdf"/>
   <xacro:wsg32_link base_link='base_link_gripper' materials_="0"/>
-  <xacro:include filename="$(find fingers_description)/fingers/sun_tactile.urdf"/>
+  <xacro:include filename="$(find sun_fingers_description_ros2)/fingers/sun_tactile.urdf"/>
   <xacro:tactile_link base_link_1='ext_finger_1' xyz_1="-0.0379 0.02 -0.0987" rpy_1="-1.5902 0.01 -1.5511" base_link_2='ext_finger_2' xyz_2="-0.0369 0.02 -0.099" rpy_2="-1.5805 0.01 -1.55"/>
 <xacro:include filename="$(find realsense2_description)/urdf/_d435i.urdf.xacro"/>

File: grippers/gripper_tactile_gazebo.xacro (robot description, xacro)
@@ -19,5 +19,5 @@
             <origin xyz="0 0 0" rpy="0 0 0"/>
             <geometry>
-                <mesh filename="file://$(find gripper_description)/meshes/base_link.stl" scale="0.001 0.001 0.001"/>
+                <mesh filename="file://$(find gripper_description_ros2)/meshes/base_link.stl" scale="0.001 0.001 0.001"/>
             </geometry>
             <material name="white1"/>
@@ -26,5 +26,5 @@
             <origin xyz="0 0 0" rpy="0 0 0"/>
             <geometry>
-                <mesh filename="file://$(find gripper_description)/meshes/base_link.stl" scale="0.001 0.001 0.001"/>
+                <mesh filename="file://$(find gripper_description_ros2)/meshes/base_link.stl" scale="0.001 0.001 0.001"/>
             </geometry>
         </collision>
@@ -39,5 +39,5 @@
           <origin xyz="-0.073096 0.106795 -0.04492" rpy="0 0 0"/>
           <geometry>
-            <mesh filename="file://$(find gripper_description)/meshes/finger_ext_1.stl" scale="0.001 0.001 0.001"/>
+            <mesh filename="file://$(find gripper_description_ros2)/meshes/finger_ext_1.stl" scale="0.001 0.001 0.001"/>
           </geometry>
           <material name="white1"/>
@@ -46,5 +46,5 @@
           <origin xyz="-0.073096 0.106795 -0.04492" rpy="0 0 0"/>
           <geometry>
-            <mesh filename="file://$(find gripper_description)/meshes/finger_ext_1.stl" scale="0.001 0.001 0.001"/>
+            <mesh filename="file://$(find gripper_description_ros2)/meshes/finger_ext_1.stl" scale="0.001 0.001 0.001"/>
           </geometry>
         </collision>
@@ -59,5 +59,5 @@
           <origin xyz="0.013389 0.107102 -0.046481" rpy="0 0 0"/>
           <geometry>
-            <mesh filename="file://$(find gripper_description)/meshes/finger_ext_2.stl" scale="0.001 0.001 0.001"/>
+            <mesh filename="file://$(find gripper_description_ros2)/meshes/finger_ext_2.stl" scale="0.001 0.001 0.001"/>
           </geometry>
           <material name="white1"/>
@@ -66,5 +66,5 @@
           <origin xyz="0.013389 0.107102 -0.046481" rpy="0 0 0"/>
           <geometry>
-            <mesh filename="file://$(find gripper_description)/meshes/finger_ext_2.stl" scale="0.001 0.001 0.001"/>
+            <mesh filename="file://$(find gripper_description_ros2)/meshes/finger_ext_2.stl" scale="0.001 0.001 0.001"/>
           </geometry>
         </collision>
@@ -80,7 +80,7 @@
         <child link="ext_finger_3"/>
       </joint>
-    <xacro:include filename="$(find wsg32_description)/grippers/wsg32.urdf"/>
+    <xacro:include filename="$(find wsg32_description_ros2)/grippers/wsg32.urdf"/>
     <xacro:wsg32_link base_link='base_link_gripper' xyz="-0.035 0.030 -0.026" rpy="${-90*deg} 0 ${-90*deg}" materials_="0"/>
-    <xacro:include filename="$(find fingers_description)/fingers/sun_tactile.urdf"/>
+    <xacro:include filename="$(find sun_fingers_description_ros2)/fingers/sun_tactile.urdf"/>
     <xacro:tactile_link base_link_1='ext_finger_1' xyz_1="0.016703 -0.035481 -0.000855" rpy_1="0 0 0" base_link_2='ext_finger_3' xyz_2="-0.016415 -0.035555 0.000618" rpy_2="0 0 0"/>
     </xacro:macro>

Commit message: add pusher with tactile sensor

File: grippers/gripper_pushing.xacro (robot description, xacro)
@@ -1,30 +1,65 @@
 <?xml version='1.0' encoding='utf-8'?>
 <robot xmlns:xacro="http://www.ros.org/wiki/xacro" name="wgs32_camera">
-    <xacro:property name="deg" value="0.017453293" /> <!--degrees to radians-->
-    <xacro:include filename="$(find gripper_description_ros2)/grippers/gripper_tactile.xacro"/>
-    <link name="push_extension">
-        <inertial>
-          <origin xyz="-0.002113007458297622 -0.026370216471355318 -0.000277269428080415" rpy="0 0 0"/>
-          <mass value="0.06014924243379804"/>
-          <inertia ixx="4.3e-05" iyy="1.7e-05" izz="2.7e-05" ixy="0.0" iyz="1.6e-05" ixz="-0.0"/>
-        </inertial>
-        <visual>
-          <origin xyz="0 0 0" rpy="0 0 0"/>
-          <geometry>
-            <mesh filename="file://$(find gripper_description_ros2)/meshes/pusher_ext.stl" scale="0.001 0.001 0.001"/>
-          </geometry>
-          <material name="white1"/>
-        </visual>
-        <collision>
-          <origin xyz="0 0 0" rpy="0 0 0"/>
-          <geometry>
-            <mesh filename="file://$(find gripper_description_ros2)/meshes/pusher_ext.stl" scale="0.001 0.001 0.001"/>
-          </geometry>
-        </collision>
-      </link>
-      <joint name="tactile_joint_pusher" type="fixed">
-        <origin xyz="0.00012757793764987647 -0.2859275779376499 0.07637889688249402" rpy="-1.5606521280013759 0.00020384840978560081 0.020189250214579735"/>
-        <parent link="tactile_2"/>
-        <child link="push_extension"/>
-      </joint>
+  <xacro:property name="deg" value="0.017453293" />
+  <!--degrees to radians-->
+  <xacro:include filename="$(find gripper_description_ros2)/grippers/gripper_tactile.xacro"/>
+  <link name="adapter_fingerside">
+    <inertial>
+      <origin xyz="0 0 0" rpy="0 0 0"/>
+      <mass value="0.06014924243379804"/>
+      <inertia ixx="4.3e-05" iyy="1.7e-05" izz="2.7e-05" ixy="0.0" iyz="1.6e-05" ixz="-0.0"/>
+    </inertial>
+    <visual>
+      <origin xyz="0 0 0" rpy="0 0 0"/>
+      <geometry>
+        <mesh filename="file://$(find gripper_description_ros2)/meshes/adapter_fingerside.stl" scale="0.001 0.001 0.001"/>
+      </geometry>
+      <material name="white1"/>
+    </visual>
+    <collision>
+      <origin xyz="0 0 0" rpy="0 0 0"/>
+      <geometry>
+        <mesh filename="file://$(find gripper_description_ros2)/meshes/adapter_fingerside.stl" scale="0.001 0.001 0.001"/>
+      </geometry>
+    </collision>
+  </link>
+  <link name="pusher_tactile">
+    <inertial>
+      <origin xyz="0 0 0" rpy="0 0 0"/>
+      <mass value="0.06014924243379804"/>
+      <inertia ixx="4.3e-05" iyy="1.7e-05" izz="2.7e-05" ixy="0.0" iyz="1.6e-05" ixz="-0.0"/>
+    </inertial>
+    <visual>
+      <origin xyz="0.0174 0.015 0.0819" rpy="0 0 0"/>
+      <geometry>
+        <mesh filename="file://$(find gripper_description_ros2)/meshes/pusher_unified_v2.stl" scale="0.001 0.001 0.001"/>
+      </geometry>
+      <material name="white1"/>
+    </visual>
+    <collision>
+      <origin xyz="0 0 0" rpy="0 0 0"/>
+      <geometry>
+        <mesh filename="file://$(find gripper_description_ros2)/meshes/pusher_unified_v2.stl" scale="0.001 0.001 0.001"/>
+      </geometry>
+    </collision>
+  </link>
+  <!-- <link name="revolute_pusher"></link> -->
+  <joint name="tactile_2_adapter" type="fixed">
+    <origin xyz="-0.0021 -0.24539999999999998 0.0358" rpy="2.034443935795705 -1.5487669913464823 -0.46364760900080837"/>
+    <parent link="tactile_2"/>
+    <child link="adapter_fingerside"/>
+  </joint>
+  <joint name="rotation_pusher" type="revolute">
+    <origin xyz="0 0 0" rpy="0.0 0.0 0.0" />
+    <parent link="adapter_fingerside" />
+    <child link="pusher_tactile" />
+    <axis xyz="0 -1 0" />
+    <limit lower="${-180.0*deg}" upper="${0*deg}" effort="0" velocity="${200.0*deg}" />
+  </joint>
+  <link name="push_extension"></link>
+  <joint name="push_fixed" type="fixed">
+    <origin xyz="0.0174 0.015 0.0819" rpy="0 0 0"/>
+    <parent link="pusher_tactile"/>
+    <child link="push_extension"/>
+  </joint>
 </robot>

File: grippers/gripper_tactile.xacro (robot description, xacro)
@@ -112,9 +112,9 @@
 </xacro:sensor_d435i> -->
 <!-- END EFFECTOR FINGERS -->
-<link name="ee_fingers"> </link>
+<!-- <link name="ee_fingers"> </link>
 <joint name="tool0_ee" type="fixed">
   <origin xyz="0 0 0.21" rpy="0 0 0"/>
   <parent link="tool0"/>
   <child link="ee_fingers"/>
-</joint>
+</joint> -->
 </robot>

Commit message: fixed revolute joint for pusher

File: grippers/gripper_pushing.xacro (robot description, xacro)
@@ -50,5 +50,5 @@
     <child link="adapter_fingerside"/>
   </joint>
-  <joint name="rotation_pusher" type="revolute">
+  <joint name="rotation_pusher" type="fixed">
     <origin xyz="0 0 0" rpy="0.0 0.0 0.0" />
     <parent link="adapter_fingerside" />

File: grippers/gripper_tactile.xacro (robot description, xacro)
@@ -112,9 +112,9 @@
 </xacro:sensor_d435i> -->
 <!-- END EFFECTOR FINGERS -->
-<!-- <link name="ee_fingers"> </link>
+<link name="ee_fingers"> </link>
 <joint name="tool0_ee" type="fixed">
   <origin xyz="0 0 0.21" rpy="0 0 0"/>
   <parent link="tool0"/>
   <child link="ee_fingers"/>
-</joint> -->
+</joint>
 </robot>
