Commit message: add materials and push extension

File: grippers/gripper_iiwa_pushing.xacro (robot description, xacro)
@@ -1,8 +1,9 @@
 <?xml version='1.0' encoding='utf-8'?>
-<robot xmlns:xacro="http://www.ros.org/wiki/xacro" name="wgs32_camera">
+<robot xmlns:xacro="http://www.ros.org/wiki/xacro" name="wgs50_push_config">
   <xacro:property name="deg" value="0.017453293" />
   <!--degrees to radians-->
   <xacro:include filename="$(find gripper_description_ros2)/grippers/gripper_iiwa_tactile.xacro"/>
-  <!-- <link name="adapter_fingerside">
+  <xacro:include filename="$(find gripper_description_ros2)/grippers/materials_.xacro"/>
+  <link name="adapter_fingerside">
     <inertial>
       <origin xyz="0 0 0" rpy="0 0 0"/>
@@ -15,5 +16,5 @@
         <mesh filename="file://$(find gripper_description_ros2)/meshes/adapter_fingerside.stl" scale="0.001 0.001 0.001"/>
       </geometry>
-      <material name="white1"/>
+      <material name="silver"/>
     </visual>
     <collision>
@@ -35,5 +36,5 @@
         <mesh filename="file://$(find gripper_description_ros2)/meshes/pusher_unified_v2.stl" scale="0.001 0.001 0.001"/>
       </geometry>
-      <material name="white1"/>
+      <material name="black"/>
     </visual>
     <collision>
@@ -44,8 +45,7 @@
     </collision>
   </link>
-  <link name="revolute_pusher"></link>
   <joint name="tactile_2_adapter" type="fixed">
     <origin xyz="-0.0021 -0.24539999999999998 0.0358" rpy="2.034443935795705 -1.5487669913464823 -0.46364760900080837"/>
-    <parent link="tactile_2"/>
+    <parent link="tactile_1"/>
     <child link="adapter_fingerside"/>
   </joint>
@@ -62,4 +62,4 @@
     <parent link="pusher_tactile"/>
     <child link="push_extension"/>
-  </joint>  -->
+  </joint>
 </robot>

File: grippers/gripper_iiwa_tactile.xacro (robot description, xacro)
@@ -1,4 +1,4 @@
 <?xml version='1.0' encoding='utf-8'?>
-<robot xmlns:xacro="http://www.ros.org/wiki/xacro" name="wgs32_camera">
+<robot xmlns:xacro="http://www.ros.org/wiki/xacro" name="wgs50_tactile_camera">
   <xacro:property name="deg" value="0.017453293" />
   <xacro:property name="base_link" value="base_link_gripper"/>
