Commit message: add contact frame

File: grippers/gripper_wsg50_pushing.xacro (robot description, xacro)
@@ -62,5 +62,5 @@
   </joint>
   <joint name="push_fixed" type="fixed">
-    <origin xyz="0.0174 0.015 0.0819" rpy="0 0 0" />
+    <origin xyz="0.0174 0.015 0.0819" rpy="1.57 0 1.57" />
     <parent link="pusher_tactile" />
     <child link="push_extension" />

Commit message: fix pusher kinematics

File: grippers/gripper_wsg50_pushing.xacro (robot description, xacro)
@@ -32,5 +32,5 @@
     </inertial>
     <visual>
-      <origin xyz="0.0174 0.015 0.0819" rpy="0 0 0" />
+      <origin xyz="0.0174 0.015 0.0819" rpy="0 0 -0.2" />
       <geometry>
         <mesh filename="file://$(find gripper_description_ros2)/meshes/pusher_unified_v2.stl"
@@ -51,4 +51,5 @@
     <origin xyz="-0.0021 -0.24539999999999998 0.0358"
       rpy="2.034443935795705 -1.5487669913464823 -0.46364760900080837" />
+      <!-- rpy="2.034443935795705 -1.5487669913464823 -0.46364760900080837" -->
     <parent link="tactile_1" />
     <child link="adapter_fingerside" />
@@ -62,5 +63,5 @@
   </joint>
   <joint name="push_fixed" type="fixed">
-    <origin xyz="0.0174 0.015 0.0819" rpy="1.57 0 1.57" />
+    <origin xyz="0.0174 0.015 0.0819" rpy="1.57 0 1.40" />
     <parent link="pusher_tactile" />
     <child link="push_extension" />

File: grippers/wsg50_tactile_camera.xacro (robot description, xacro)
@@ -18,5 +18,5 @@
   <xacro:tactile_link base_link_1="${prefix_finger_right}${finger_flange_link}"
     xyz_1="-0.0127 -0.0361 -0.0535"
-    rpy_1="-1.57 0.0 0.02" base_link_2='${prefix_finger_left}${finger_flange_link}'
+    rpy_1="-1.57 0.0 0.10" base_link_2='${prefix_finger_left}${finger_flange_link}'
     xyz_2="-0.0127 -0.0361 -0.0535"
     rpy_2="-1.57 0 0.02" />

Commit message: update transformation camera robot

File: grippers/gripper_wsg50_pushing.xacro (robot description, xacro)
@@ -63,5 +63,5 @@
   </joint>
   <joint name="push_fixed" type="fixed">
-    <origin xyz="0.0174 0.015 0.0819" rpy="1.57 0 1.40" />
+    <origin xyz="0.0174 0.015 0.0819" rpy="1.57 0 1.43" />
     <parent link="pusher_tactile" />
     <child link="push_extension" />

File: grippers/wsg50_tactile_camera_ext.xacro (robot description, xacro)
@@ -45,5 +45,5 @@
   </link>
   <joint name="camera_ext_joint" type="fixed">
-    <origin xyz="0 -0.04 0.0006" rpy="-1.57 0 -3.140" />
+    <origin xyz="0 -0.004 0.0006" rpy="-1.65 0 -3.140" />
     <parent link="${base_link}" />
     <child link="camera_ext" />
@@ -52,6 +52,8 @@
   <xacro:include filename="$(find realsense2_description)/urdf/_d435i.urdf.xacro" />
   <xacro:sensor_d435i parent="camera_ext" name="camera" use_nominal_extrinsics="true">
+    <!-- without extension -->
     <!-- <origin xyz="-0.0322 0.0895 -0.0325" rpy="0 -1.30899694 -1.57" /> -->
-    <origin xyz="-0.033 0.0795 0.1498" rpy="0   0.14   -1.5700" />
+    <!-- with extension -->
+    <origin xyz="-0.033 0.0795 0.1498" rpy="0   0.1   -1.55" />
   </xacro:sensor_d435i>
   <!-- -0.0322 0.0895 -0.0325 0 -1.30899694 -1.57 -->

Commit message: fixed xacro

File: grippers/gripper_wsg50_pushing.xacro (robot description, xacro)
@@ -32,5 +32,5 @@
     </inertial>
     <visual>
-      <origin xyz="0.0174 0.015 0.0819" rpy="0 0 -0.2" />
+      <origin xyz="0.0174 0.015 0.0819" rpy="0 0 0" />
       <geometry>
         <mesh filename="file://$(find gripper_description_ros2)/meshes/pusher_unified_v2.stl"
@@ -63,5 +63,5 @@
   </joint>
   <joint name="push_fixed" type="fixed">
-    <origin xyz="0.0174 0.015 0.0819" rpy="1.57 0 1.43" />
+    <origin xyz="0.0174 0.015 0.0819" rpy="1.57 0 1.48" />
     <parent link="pusher_tactile" />
     <child link="push_extension" />

File: grippers/wsg50_tactile_camera_ext.xacro (robot description, xacro)
@@ -45,5 +45,5 @@
   </link>
   <joint name="camera_ext_joint" type="fixed">
-    <origin xyz="0 -0.004 0.0006" rpy="-1.65 0 -3.140" />
+    <origin xyz="0.005 0.0 0.0006" rpy="-1.65 0 -3.140" />
     <parent link="${base_link}" />
     <child link="camera_ext" />
@@ -55,5 +55,5 @@
     <!-- <origin xyz="-0.0322 0.0895 -0.0325" rpy="0 -1.30899694 -1.57" /> -->
     <!-- with extension -->
-    <origin xyz="-0.033 0.0795 0.1498" rpy="0   0.1   -1.55" />
+    <origin xyz="-0.030 0.0795 0.1498" rpy="0   0.1   -1.55" />
   </xacro:sensor_d435i>
   <!-- -0.0322 0.0895 -0.0325 0 -1.30899694 -1.57 -->
